File: Hardware/SparkFun_Tri_Axis_Accel_Breakout-H3LIS331DL.sch (EAGLE design)
At the start: 23 parts, among them U1 H3LIS331DL

Commit message: Aesthetic touch ups before review
Other:
- note added: "Accelerometer"
- note added: "Bypass Capacitance"
- note added: "Headers"
- note added: "Passives"
- moved on the sheet: C1, C2, J1, J2, JP1, JP2, JP3, R1, R2, R3, R4, U1

Commit message: Replace some components with newer versions
Parts:
- C1: device SparkFun:CAP_POL1206 -> SparkFun-Capacitors:10UF-POLAR-EIA3216-16V-10%(TANT)
- C2: device SparkFun:CAP0402-CAP -> SparkFun-Capacitors:0.1UF-0603-25V-5%
Changed lines of the file:
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@@
 </classes>
 <parts>
-<part name="C2" library="SparkFun" deviceset="CAP" device="0402-CAP" value="0.1uF"/>
+<part name="C2" library="SparkFun-Capacitors" deviceset="0.1UF" device="-0603-25V-5%" value="0.1uF"/>
 <part name="GND1" library="SparkFun" deviceset="GND" device=""/>
 <part name="GND5" library="SparkFun" deviceset="GND" device=""/>
 <part name="U1" library="SparkFun-Sensors" deviceset="H3LIS331DL" device="" value="H3LIS331DL"/>
 <part name="GND2" library="SparkFun" deviceset="GND" device=""/>
-<part name="C1" library="SparkFun" deviceset="CAP_POL" device="1206" value="10uF"/>
+<part name="C1" library="SparkFun-Capacitors" deviceset="10UF-POLAR" device="-EIA3216-16V-10%(TANT)" value="10uF"/>
 <part name="JP11" library="SparkFun" deviceset="STAND-OFF" device=""/>
 <part name="JP10" library="SparkFun" deviceset="STAND-OFF" device=""/>

Commit message: Modified I2C address jumper note
Other:
- note added: "JP2 selects LSB of I2C address Open Addr= 0x19 Closed Addr=0x18"
- note removed: "JP2 selects LSB of I2C address"
Changed lines of the file:
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@@
 pull-up resistors</text>
 <text x="205.74" y="104.14" size="1.778" layer="94">JP2 selects LSB
-of I2C address</text>
+of I2C address
+Open Addr= 0x19
+Closed Addr=0x18</text>
 <text x="190.5" y="86.36" size="1.778" layer="94">Clear JP3 to enable SPI mode</text>
 <wire x1="147.32" y1="35.56" x2="147.32" y2="63.5" width="0.3048" layer="97" style="longdash"/>

Commit message: Improvements post review
Other:
- note added: "10"
- note added: "2.16V < VCC < 3.6V"
- note removed: "01"
Changed lines of the file:
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@@
 <plain>
 <text x="172.72" y="7.62" size="3.81" layer="94">Mike Hord</text>
-<text x="239.268" y="6.096" size="3.81" layer="94">01</text>
+<text x="239.268" y="6.096" size="3.81" layer="94">10</text>
 <text x="165.1" y="134.62" size="1.778" layer="94">Open JP1 to eliminate
 pull-up resistors</text>
@@
 <text x="83.82" y="55.88" size="3.81" layer="97">Bypass Capacitance</text>
 <text x="149.86" y="38.1" size="3.81" layer="97">Passives</text>
+<text x="78.74" y="147.32" size="2.54" layer="97">2.16V &lt; VCC &lt; 3.6V</text>
 </plain>
 <instances>
